Commit message: reset function

File: mm-walker/mm_walker/envs/urdf/robot.urdf (robot description, URDF)
Before this commit: robot robot, 9 links, 8 joints
Links:
- link corpus: geometry collision mesh filename=../mesh/Corpus.stl scale=0.01 0.01 0.01; visual mesh filename=../mesh/Corpus.stl scale=0.01 0.01 0.01
- link foot_front_left: geometry collision mesh filename=../mesh/FootL.stl scale=0.01 0.01 0.01; visual mesh filename=../mesh/FootL.stl scale=0.01 0.01 0.01
- link foot_front_right: geometry collision mesh filename=../mesh/FootR.stl scale=0.01 0.01 0.01; visual mesh filename=../mesh/FootR.stl scale=0.01 0.01 0.01
- link foot_rear_left: geometry collision mesh filename=../mesh/FootR.stl scale=0.01 0.01 0.01; visual mesh filename=../mesh/FootR.stl scale=0.01 0.01 0.01
- link foot_rear_right: geometry collision mesh filename=../mesh/FootL.stl scale=0.01 0.01 0.01; visual mesh filename=../mesh/FootL.stl scale=0.01 0.01 0.01
- link upper_leg_front_left: geometry collision mesh filename=../mesh/UpperLegL.stl scale=0.01 0.01 0.01; visual mesh filename=../mesh/UpperLegL.stl scale=0.01 0.01 0.01
- link upper_leg_front_right: geometry collision mesh filename=../mesh/UpperLegR.stl scale=0.01 0.01 0.01; visual mesh filename=../mesh/UpperLegR.stl scale=0.01 0.01 0.01
- link upper_leg_rear_left: geometry collision mesh filename=../mesh/UpperLegR.stl scale=0.01 0.01 0.01; visual mesh filename=../mesh/UpperLegR.stl scale=0.01 0.01 0.01
- link upper_leg_rear_right: geometry collision mesh filename=../mesh/UpperLegL.stl scale=0.01 0.01 0.01; visual mesh filename=../mesh/UpperLegL.stl scale=0.01 0.01 0.01

Commit message: Action control frequency

File: mm-walker/mm_walker/envs/urdf/robot.urdf (robot description, URDF)
Before this commit: robot robot, 9 links, 8 joints
Joints:
- joint upper_leg_to_foot_rr: limit lower=-1,9 upper=2.2 effort=93000 velocity=5.1 -> lower=-1.9 upper=2.2 effort=93000 velocity=5.1

Commit message: Walking real robot 5Hz Increased weight

File: mm-walker/mm_walker/envs/urdf/robot.urdf (robot description, URDF)
Before this commit: robot robot, 9 links, 8 joints
Links:
- link corpus: mass 561 -> 750
